Commit message: update

File: description/imu.xacro (robot description, xacro)
@@ -2,15 +2,9 @@
 <robot xmlns:xacro="http://ros.org/wiki/xacro">
     <!-- Imu sensor  -->
-    <link name="imu_link">
-        <visual name="imu_visual">
-            <geometry>
-                <mesh filename="package://agvbot_pro/model/mpu6050.dae" />
-            </geometry>
-        </visual>
-    </link>
+    <link name="imu_link"></link>
     <joint name="imu_joint" type="fixed">
         <parent link="chassis" />
         <child link="imu_link" />
-        <origin xyz="0.15 0 0" rpy="0 ${pi} ${pi/2}" />
+        <origin xyz="0.35 0 0" rpy="0 ${pi} ${pi/2}" />
     </joint>
     <gazebo reference="imu_link">

File: description/lidar.xacro (robot description, xacro)
@@ -4,5 +4,5 @@
         <parent link="chassis" />
         <child link="laser_frame" />
-        <origin xyz="0.15 0 0.14" rpy="0 0 0" />
+        <origin xyz="0.35 0 0.17" rpy="0 0 0" />
     </joint>
     <link name="laser_frame">

File: description/robot_core.xacro (robot description, xacro)
@@ -2,13 +2,13 @@
 <robot xmlns:xacro="http://www.ros.org/wiki/xacro">
     <xacro:include filename="inertial_macros.xacro" />
-    <xacro:property name="chassis_length" value="0.30" />
-    <xacro:property name="chassis_width" value="0.30" />
-    <xacro:property name="chassis_height" value="0.085" />
+    <xacro:property name="chassis_length" value="0.70" />
+    <xacro:property name="chassis_width" value="0.60" />
+    <xacro:property name="chassis_height" value="0.126" />
     <xacro:property name="chassis_mass" value="1.5" />
-    <xacro:property name="wheel_radius" value="0.0325" />
-    <xacro:property name="wheel_thickness" value="0.027" />
+    <xacro:property name="wheel_radius" value="0.05" />
+    <xacro:property name="wheel_thickness" value="0.04" />
     <xacro:property name="wheel_mass" value="0.05" />
-    <xacro:property name="wheel_offset_x" value="0.15" />
-    <xacro:property name="wheel_offset_y" value="0.13" />
+    <xacro:property name="wheel_offset_x" value="0.35" />
+    <xacro:property name="wheel_offset_y" value="0.205" />
     <xacro:property name="wheel_offset_z" value="-0.02" />
     <xacro:property name="caster_wheel_radius" value="0.01" />
@@ -17,9 +17,4 @@
     <xacro:property name="caster_wheel_offset_z"
         value="${wheel_offset_z - wheel_radius + caster_wheel_radius}" />
-    <xacro:property name="caster1_wheel_radius" value="0.01" />
-    <xacro:property name="caster1_wheel_mass" value="0.1" />
-    <xacro:property name="caster1_wheel_offset_x" value="0.28" />
-    <xacro:property name="caster1_wheel_offset_z"
-        value="${wheel_offset_z - wheel_radius + caster1_wheel_radius}" />
     <material name="white">
         <color rgba="1 1 1 1" />
@@ -131,49 +126,23 @@
     </gazebo>
     <!-- CASTER WHEEL LINK -->
-    <joint name="caster_wheel_joint" type="fixed">
-        <parent link="chassis" />
-        <child link="caster_wheel" />
-        <origin xyz="${caster_wheel_offset_x} 0 ${caster_wheel_offset_z}" />
-    </joint>
-    <link name="caster_wheel">
-        <visual>
-            <geometry>
-                <sphere radius="${caster_wheel_radius}" />
-            </geometry>
-            <material name="blue" />
-        </visual>
-        <collision>
-            <geometry>
-                <sphere radius="${caster_wheel_radius}" />
-            </geometry>
-        </collision>
-        <xacro:inertial_sphere mass="${caster_wheel_mass}" radius="${caster_wheel_radius}">
-            <origin xyz="0 0 0" rpy="0 0 0" />
-        </xacro:inertial_sphere>
-    </link>
-    <gazebo reference="caster_wheel">
-        <material>Gazebo/Blue</material>
-        <mu1 value="0.001" />
-        <mu2 value="0.001" />
-    </gazebo>
-    <!-- CASTER1 WHEEL LINK -->
+    <!-- WHEEL LINK == 1 -->
     <joint name="caster1_wheel_joint" type="fixed">
         <parent link="chassis" />
         <child link="caster1_wheel" />
-        <origin xyz="${caster1_wheel_offset_x} 0 ${caster1_wheel_offset_z}" />
+        <origin xyz="0.05 0.2 ${caster_wheel_offset_z}" />
     </joint>
     <link name="caster1_wheel">
         <visual>
             <geometry>
-                <sphere radius="${caster1_wheel_radius}" />
-            </geometry>
-            <material name="blue" />
-        </visual>
-        <collision>
-            <geometry>
-                <sphere radius="${caster1_wheel_radius}" />
-            </geometry>
-        </collision>
-        <xacro:inertial_sphere mass="${caster1_wheel_mass}" radius="${caster1_wheel_radius}">
+                <sphere radius="${caster_wheel_radius}" />
+            </geometry>
+            <material name="blue" />
+        </visual>
+        <collision>
+            <geometry>
+                <sphere radius="${caster_wheel_radius}" />
+            </geometry>
+        </collision>
+        <xacro:inertial_sphere mass="${caster_wheel_mass}" radius="${caster_wheel_radius}">
             <origin xyz="0 0 0" rpy="0 0 0" />
         </xacro:inertial_sphere>
@@ -184,3 +153,84 @@
         <mu2 value="0.001" />
     </gazebo>
+    <!-- WHEEL LINK == 2 -->
+    <joint name="caster2_wheel_joint" type="fixed">
+        <parent link="chassis" />
+        <child link="caster2_wheel" />
+        <origin xyz="0.05 -0.2 ${caster_wheel_offset_z}" />
+    </joint>
+    <link name="caster2_wheel">
+        <visual>
+            <geometry>
+                <sphere radius="${caster_wheel_radius}" />
+            </geometry>
+            <material name="blue" />
+        </visual>
+        <collision>
+            <geometry>
+                <sphere radius="${caster_wheel_radius}" />
+            </geometry>
+        </collision>
+        <xacro:inertial_sphere mass="${caster_wheel_mass}" radius="${caster_wheel_radius}">
+            <origin xyz="0 0 0" rpy="0 0 0" />
+        </xacro:inertial_sphere>
+    </link>
+    <gazebo reference="caster2_wheel">
+        <material>Gazebo/Blue</material>
+        <mu1 value="0.001" />
+        <mu2 value="0.001" />
+    </gazebo>
+    <!-- WHEEL LINK == 3 -->
+    <joint name="caster3_wheel_joint" type="fixed">
+        <parent link="chassis" />
+        <child link="caster3_wheel" />
+        <origin xyz="0.65 -0.2 ${caster_wheel_offset_z}" />
+    </joint>
+    <link name="caster3_wheel">
+        <visual>
+            <geometry>
+                <sphere radius="${caster_wheel_radius}" />
+            </geometry>
+            <material name="blue" />
+        </visual>
+        <collision>
+            <geometry>
+                <sphere radius="${caster_wheel_radius}" />
+            </geometry>
+        </collision>
+        <xacro:inertial_sphere mass="${caster_wheel_mass}" radius="${caster_wheel_radius}">
+            <origin xyz="0 0 0" rpy="0 0 0" />
+        </xacro:inertial_sphere>
+    </link>
+    <gazebo reference="caster3_wheel">
+        <material>Gazebo/Blue</material>
+        <mu1 value="0.001" />
+        <mu2 value="0.001" />
+    </gazebo>
+    <!-- WHEEL LINK == 4 -->
+    <joint name="caster4_wheel_joint" type="fixed">
+        <parent link="chassis" />
+        <child link="caster4_wheel" />
+        <origin xyz="0.65 0.2 ${caster_wheel_offset_z}" />
+    </joint>
+    <link name="caster4_wheel">
+        <visual>
+            <geometry>
+                <sphere radius="${caster_wheel_radius}" />
+            </geometry>
+            <material name="blue" />
+        </visual>
+        <collision>
+            <geometry>
+                <sphere radius="${caster_wheel_radius}" />
+            </geometry>
+        </collision>
+        <xacro:inertial_sphere mass="${caster_wheel_mass}" radius="${caster_wheel_radius}">
+            <origin xyz="0 0 0" rpy="0 0 0" />
+        </xacro:inertial_sphere>
+    </link>
+    <gazebo reference="caster4_wheel">
+        <material>Gazebo/Blue</material>
+        <mu1 value="0.001" />
+        <mu2 value="0.001" />
+    </gazebo>
 </robot>

File: description/ros2_control.xacro (robot description, xacro)
@@ -8,9 +8,9 @@
                 <param name="left_wheel_name">left_wheel_joint</param>
                 <param name="right_wheel_name">right_wheel_joint</param>
-                <param name="loop_rate">20</param>
-                <param name="device">/dev/ttyUSB1</param>
+                <param name="loop_rate">30</param>
+                <param name="device">/dev/serial/by-path/platform-fd500000.pcie-pci-0000:01:00.0-usb-0:1.1:1.0</param>
                 <param name="baud_rate">57600</param>
                 <param name="timeout">1000</param>
-                <param name="enc_counts_per_rev">1320</param>
+                <param name="enc_counts_per_rev">200</param>
             </hardware>
             <joint name="left_wheel_joint">
@@ -32,5 +32,5 @@
         </ros2_control>
         <!-- MPU6050 sensor-->
-        <ros2_control name='MPU6050' type='sensor'>
+        <!-- <ros2_control name='MPU6050' type='sensor'>
             <hardware>
                 <plugin>lidarbot_bringup/MPU6050Hardware</plugin>
@@ -50,5 +50,5 @@
                 <state_interface name='linear_acceleration.z' />
             </sensor>
-        </ros2_control>
+        </ros2_control> -->
     </xacro:unless>
     <xacro:if value="$(arg sim_mode)">
