Commit message: update

File: description/robot_core.xacro (robot description, xacro)
@@ -2,19 +2,18 @@
 <robot xmlns:xacro="http://www.ros.org/wiki/xacro">
     <xacro:include filename="inertial_macros.xacro" />
-    <xacro:property name="chassis_length" value="0.70" />
-    <xacro:property name="chassis_width" value="0.60" />
-    <xacro:property name="chassis_height" value="0.126" />
-    <xacro:property name="chassis_mass" value="1.5" />
-    <xacro:property name="wheel_radius" value="0.05" />
-    <xacro:property name="wheel_thickness" value="0.04" />
-    <xacro:property name="wheel_mass" value="0.05" />
-    <xacro:property name="wheel_offset_x" value="0.35" />
-    <xacro:property name="wheel_offset_y" value="0.205" />
-    <xacro:property name="wheel_offset_z" value="-0.02" />
-    <xacro:property name="caster_wheel_radius" value="0.01" />
-    <xacro:property name="caster_wheel_mass" value="0.1" />
-    <xacro:property name="caster_wheel_offset_x" value="0.02" />
-    <xacro:property name="caster_wheel_offset_z"
-        value="${wheel_offset_z - wheel_radius + caster_wheel_radius}" />
+    <xacro:property name="chassis_length"   value="0.70" />
+    <xacro:property name="chassis_width"    value="0.60" />
+    <xacro:property name="chassis_height"   value="0.126" />
+    <xacro:property name="chassis_mass"     value="1.5" />
+    <xacro:property name="wheel_radius"     value="0.05" />
+    <xacro:property name="wheel_thickness"  value="0.04" />
+    <xacro:property name="wheel_mass"       value="0.05" />
+    <xacro:property name="wheel_offset_x"   value="0.35" />
+    <xacro:property name="wheel_offset_y"   value="0.205" />
+    <xacro:property name="wheel_offset_z"   value="-0.02" />
+    <xacro:property name="caster_wheel_radius"      value="0.01" />
+    <xacro:property name="caster_wheel_mass"        value="0.1" />
+    <xacro:property name="caster_wheel_offset_x"    value="0.02" />
+    <xacro:property name="caster_wheel_offset_z"    value="${wheel_offset_z - wheel_radius + caster_wheel_radius}" />
     <material name="white">
         <color rgba="1 1 1 1" />
@@ -55,5 +54,5 @@
                 <box size="${chassis_length} ${chassis_width} ${chassis_height}" />
             </geometry>
-            <material name="white" />
+            <material name="orange" />
         </visual>
         <collision>
@@ -69,5 +68,5 @@
     </link>
     <gazebo reference="chassis">
-        <material>Gazebo/White</material>
+        <material>Gazebo/Orange</material>
     </gazebo>
     <!-- LEFT WHEEL LINK -->
